File: Board.brd (EAGLE design)
At the start: 100 x 80 mm, 26 parts, among them X1 1503_02

Commit message: updated library pads position to go a bit under the module so they can be soldered easier
Changed lines of the file:
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@@
 <contactref element="C1" pad="1"/>
 <contactref element="U$1" pad="MIC_P"/>
-<wire x1="47.32" y1="62.98" x2="50.15" y2="62.98" width="0.8" layer="1"/>
+<wire x1="47.22" y1="62.98" x2="50.15" y2="62.98" width="0.8" layer="1"/>
 <wire x1="50.15" y1="62.98" x2="50.15" y2="58" width="0.8" layer="1"/>
 <wire x1="50.15" y1="58" x2="52.76" y2="58" width="0.8" layer="1"/>
@@
 <wire x1="49.05" y1="56.28" x2="49.05" y2="61.8" width="0.8" layer="1"/>
 <wire x1="49.05" y1="61.8" x2="47.32" y2="61.8" width="0.8" layer="1"/>
-<wire x1="47.32" y1="61.8" x2="47.32" y2="61.88" width="0.8" layer="1"/>
+<wire x1="47.32" y1="61.8" x2="47.22" y2="61.88" width="0.8" layer="1"/>
 </signal>
 <signal name="MIC_BIAS">
@@
 <wire x1="51.25" y1="61.75" x2="51.25" y2="64.05" width="0.8" layer="1"/>
 <wire x1="51.25" y1="64.05" x2="47.32" y2="64.05" width="0.8" layer="1"/>
-<wire x1="47.32" y1="64.05" x2="47.32" y2="64.08" width="0.8" layer="1"/>
+<wire x1="47.32" y1="64.05" x2="47.22" y2="64.08" width="0.8" layer="1"/>
 </signal>
 <signal name="N$6">
@@
 <contactref element="C8" pad="2"/>
 <contactref element="C9" pad="2"/>
-<wire x1="47.32" y1="73.98" x2="50.48" y2="73.98" width="0.8" layer="1"/>
+<wire x1="47.22" y1="73.98" x2="50.48" y2="73.98" width="0.8" layer="1"/>
 <wire x1="50.72" y1="71.4" x2="53.31" y2="71.4" width="0.8" layer="1"/>
 <wire x1="50.72" y1="71.4" x2="50.71" y2="71.41" width="0.8" layer="1"/>
 <wire x1="50.71" y1="71.41" x2="50.71" y2="73.75" width="0.8" layer="1"/>
 <wire x1="50.71" y1="73.75" x2="50.48" y2="73.98" width="0.8" layer="1"/>
-<wire x1="34.15" y1="73.98" x2="32.22" y2="73.98" width="0.8" layer="1"/>
+<wire x1="34.15" y1="73.98" x2="32.32" y2="73.98" width="0.8" layer="1"/>
 <contactref element="POWER" pad="1"/>
 <wire x1="34.15" y1="73.98" x2="42.2" y2="73.98" width="0.8" layer="1"/>
-<wire x1="42.2" y1="73.98" x2="47.32" y2="73.98" width="0.8" layer="1"/>
+<wire x1="42.2" y1="73.98" x2="47.22" y2="73.98" width="0.8" layer="1"/>
 <wire x1="34.15" y1="73.98" x2="34.15" y2="71.8" width="0.8" layer="1"/>
 <wire x1="34.15" y1="71.8" x2="32.22" y2="71.8" width="0.8" layer="1"/>
-<wire x1="32.22" y1="71.8" x2="32.22" y2="71.78" width="0.8" layer="1"/>
-<wire x1="32.22" y1="73.98" x2="30.65" y2="73.98" width="0.8" layer="1"/>
+<wire x1="32.22" y1="71.8" x2="32.32" y2="71.78" width="0.8" layer="1"/>
+<wire x1="32.32" y1="73.98" x2="30.65" y2="73.98" width="0.8" layer="1"/>
 <wire x1="30.65" y1="73.98" x2="30.65" y2="74" width="0.8" layer="1"/>
 <wire x1="30.65" y1="74" x2="29.8" y2="74.85" width="0.8" layer="1"/>
@@
 <wire x1="33.8" y1="55.65" x2="33.7" y2="57.45" width="0.8" layer="1"/>
 <wire x1="33.7" y1="57.45" x2="32.22" y2="57.45" width="0.8" layer="1"/>
-<wire x1="32.22" y1="57.45" x2="32.22" y2="57.48" width="0.8" layer="1"/>
+<wire x1="32.22" y1="57.45" x2="32.32" y2="57.48" width="0.8" layer="1"/>
 <wire x1="22.45" y1="60.2" x2="22.45" y2="54.55" width="0.8" layer="1"/>
 <wire x1="24.04" y1="55.16" x2="24.2923875" y2="55.16" width="0.8" layer="1"/>
@@
 <wire x1="42.2" y1="73.98" x2="42.1" y2="73.93" width="0.8" layer="1"/>
 <wire x1="47.32" y1="57.45" x2="42.1" y2="57.4" width="0.8" layer="1"/>
-<wire x1="47.32" y1="57.45" x2="47.32" y2="57.48" width="0.8" layer="1"/>
+<wire x1="47.32" y1="57.45" x2="47.22" y2="57.48" width="0.8" layer="1"/>
 <wire x1="42.1" y1="73.93" x2="42.1" y2="57.4" width="0.8" layer="1"/>
 <wire x1="61.27" y1="58.2" x2="61.3" y2="58.2" width="0.8" layer="1"/>
@@
 <wire x1="28.5" y1="59.98" x2="28.5" y2="60.75" width="0.8" layer="1"/>
 <wire x1="28.5" y1="60.75" x2="32.22" y2="60.75" width="0.8" layer="1"/>
-<wire x1="32.22" y1="60.75" x2="32.22" y2="60.78" width="0.8" layer="1"/>
+<wire x1="32.22" y1="60.75" x2="32.32" y2="60.78" width="0.8" layer="1"/>
 </signal>
 <signal name="LED1">
@@
 <wire x1="30.3" y1="57.68" x2="30.3" y2="59.65" width="0.8" layer="1"/>
 <wire x1="30.3" y1="59.65" x2="32.22" y2="59.65" width="0.8" layer="1"/>
-<wire x1="32.22" y1="59.65" x2="32.22" y2="59.68" width="0.8" layer="1"/>
+<wire x1="32.22" y1="59.65" x2="32.32" y2="59.68" width="0.8" layer="1"/>
 </signal>
 <signal name="RP">
@@
 <wire x1="55.6" y1="62.85" x2="55.6" y2="67.4" width="0.8" layer="1"/>
 <wire x1="55.6" y1="67.4" x2="47.32" y2="67.4" width="0.8" layer="1"/>
-<wire x1="47.32" y1="67.4" x2="47.32" y2="67.38" width="0.8" layer="1"/>
+<wire x1="47.32" y1="67.4" x2="47.22" y2="67.38" width="0.8" layer="1"/>
 </signal>
 <signal name="R">
@@
 <contactref element="C7" pad="-"/>
 <contactref element="U$1" pad="LP"/>
-<wire x1="47.32" y1="66.28" x2="49.05" y2="66.28" width="0.8" layer="1"/>
+<wire x1="47.22" y1="66.28" x2="49.05" y2="66.28" width="0.8" layer="1"/>
 <wire x1="49.05" y1="66.28" x2="49.05" y2="66.3" width="0.8" layer="1"/>
 <wire x1="49.05" y1="66.3" x2="49.1" y2="66.3" width="0.8" layer="1"/>
@@
 <contactref element="U$1" pad="LN"/>
 <contactref element="U$1" pad="RN"/>
-<wire x1="45.55" y1="68.48" x2="47.32" y2="68.48" width="0.8" layer="1"/>
+<wire x1="45.55" y1="68.48" x2="47.22" y2="68.48" width="0.8" layer="1"/>
 <wire x1="45.55" y1="68.48" x2="45.55" y2="68.45" width="0.8" layer="1"/>
 <wire x1="45.55" y1="68.45" x2="45.5" y2="68.45" width="0.8" layer="1"/>
 <wire x1="45.5" y1="68.45" x2="45.5" y2="65.2" width="0.8" layer="1"/>
 <wire x1="45.5" y1="65.2" x2="47.32" y2="65.2" width="0.8" layer="1"/>
-<wire x1="47.32" y1="65.2" x2="47.32" y2="65.18" width="0.8" layer="1"/>
-<wire x1="47.32" y1="68.48" x2="57.6" y2="68.48" width="0.8" layer="1"/>
+<wire x1="47.32" y1="65.2" x2="47.22" y2="65.18" width="0.8" layer="1"/>
+<wire x1="47.22" y1="68.48" x2="57.6" y2="68.48" width="0.8" layer="1"/>
 <wire x1="57.6" y1="68.48" x2="57.6" y2="68.5" width="0.8" layer="1"/>
 </signal>
@@
 <wire x1="30.1" y1="72.6" x2="30.1" y2="64.1" width="0.8" layer="1"/>
 <wire x1="30.1" y1="64.1" x2="32.2" y2="64.1" width="0.8" layer="1"/>
-<wire x1="32.2" y1="64.1" x2="32.22" y2="64.08" width="0.8" layer="1"/>
+<wire x1="32.2" y1="64.1" x2="32.32" y2="64.08" width="0.8" layer="1"/>
 </signal>
 <signal name="RX">
@@
 <wire x1="28.6" y1="70.65" x2="28.6" y2="63" width="0.8" layer="1"/>
 <wire x1="28.6" y1="63" x2="32.22" y2="63" width="0.8" layer="1"/>
-<wire x1="32.22" y1="63" x2="32.22" y2="62.98" width="0.8" layer="1"/>
+<wire x1="32.22" y1="63" x2="32.32" y2="62.98" width="0.8" layer="1"/>
 </signal>
 <signal name="VOL+">
@@
 <wire x1="40.5" y1="54.5" x2="40.5" y2="70.65" width="0.8" layer="1"/>
 <wire x1="40.5" y1="70.65" x2="32.22" y2="70.65" width="0.8" layer="1"/>
-<wire x1="32.22" y1="70.65" x2="32.22" y2="70.68" width="0.8" layer="1"/>
+<wire x1="32.22" y1="70.65" x2="32.32" y2="70.68" width="0.8" layer="1"/>
 </signal>
 <signal name="VOL-">
@@
 <wire x1="39.22" y1="69.53" x2="39.25" y2="69.55" width="0.8" layer="1"/>
 <wire x1="39.25" y1="69.55" x2="32.25" y2="69.55" width="0.8" layer="1"/>
-<wire x1="32.25" y1="69.55" x2="32.22" y2="69.58" width="0.8" layer="1"/>
+<wire x1="32.25" y1="69.55" x2="32.32" y2="69.58" width="0.8" layer="1"/>
 </signal>
 <signal name="NEXT">
@@
 <wire x1="37.37" y1="68.43" x2="37.3" y2="68.5" width="0.8" layer="1"/>
 <wire x1="37.3" y1="68.5" x2="32.24" y2="68.5" width="0.8" layer="1"/>
-<wire x1="32.24" y1="68.5" x2="32.22" y2="68.48" width="0.8" layer="1"/>
+<wire x1="32.24" y1="68.5" x2="32.32" y2="68.48" width="0.8" layer="1"/>
 </signal>
 <signal name="PREV">
@@
 <wire x1="36.2" y1="67.35" x2="36.25" y2="67.4" width="0.8" layer="1"/>
 <wire x1="36.25" y1="67.4" x2="32.24" y2="67.4" width="0.8" layer="1"/>
-<wire x1="32.24" y1="67.4" x2="32.22" y2="67.38" width="0.8" layer="1"/>
+<wire x1="32.24" y1="67.4" x2="32.32" y2="67.38" width="0.8" layer="1"/>
 <wire x1="29.01" y1="52.94" x2="22.61" y2="52.94" width="0.8" layer="1"/>
 </signal>
@@
 <wire x1="26.65" y1="68.3" x2="26.65" y2="61.9" width="0.8" layer="1"/>
 <wire x1="26.65" y1="61.9" x2="32.22" y2="61.9" width="0.8" layer="1"/>
-<wire x1="32.22" y1="61.9" x2="32.22" y2="61.88" width="0.8" layer="1"/>
+<wire x1="32.22" y1="61.9" x2="32.32" y2="61.88" width="0.8" layer="1"/>
 </signal>
 <signal name="V3.3_SO">
@@
 <contactref element="C8" pad="1"/>
 <contactref element="C9" pad="1"/>
-<wire x1="47.32" y1="70.68" x2="49.17" y2="70.68" width="0.8" layer="1"/>
+<wire x1="47.22" y1="70.68" x2="49.17" y2="70.68" width="0.8" layer="1"/>
 <wire x1="49.17" y1="70.68" x2="49.2" y2="70.65" width="0.8" layer="1"/>
 <wire x1="49.2" y1="70.65" x2="49.2" y2="69.7" width="0.8" layer="1"/>
